File: motor_board.kicad_pcb (KiCad board)
At the start: 2 copper layers, 100 x 94.2 mm, 31 parts, among them J1 MyRIO_C, J10 ESCON_24-2, J11 Conn_01x02, J12 Conn_01x05, J13 Conn_01x03, J2 BNC, J3 BNC, J4 BNC, J5 Conn_01x04, J6 Barrel_Jack_Switch, J7 Conn_01x08, J8 Conn_01x05, J9 Conn_01x05, SW1 SW_Push, SW2 SW_Push

Commit message: the first version produced
Parts:
- added J14: BNC, motor_board:Vertical_BNC_Amphenol_112536, F.Cu at (47.1, 46.1)
- added J15: BNC, motor_board:Vertical_BNC_Amphenol_112536, F.Cu at (70.2, 46.1)
- added J16: BNC, motor_board:Vertical_BNC_Amphenol_112536, F.Cu at (93.2, 46.1)
- J2, J3, J4: footprint Connector_Coaxial:BNC_Amphenol_B6252HB-NPP3G-50_Horizontal -> motor_board:Vertical_BNC_Molex_73131-5003
- moved J5 5.77 mm to (121.0, 42.8)
- moved J6 5.77 mm to (132.2, 51.5)
- moved J2 5.76 mm to (46.8, 50.2)
- moved J3 5.76 mm to (69.8, 50.2)
- moved J4 5.76 mm to (92.8, 50.2)
Routing:
- net /AI0-: track 80.2 -> 110.1 mm
- net /AO1: track 90.7 -> 100.9 mm
- net /AI0+: track 69.2 -> 79.4 mm
- net /PWM: track 120.4 -> 127.6 mm
- net VBUS: track 27.0 -> 32.6 mm
Other:
- board size 100 x 94.2 mm -> 100 x 100 mm
