File: motor_board.kicad_pcb (KiCad board)
At the start: 2 copper layers, 100 x 100 mm, 44 parts, among them J1 MyRIO_C, J10 ESCON_24-2, J11 Conn_01x02, J12 Conn_01x05, J13 Conn_01x03, J14 BNC, J15 BNC, J2 BNC, J3 BNC, J4 BNC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

Commit message: The final design
Parts:
- C1: footprint Resistor_THT:R_Axial_DIN0204_L3.6mm_D1.6mm_P5.08mm_Horizontal -> Capacitor_THT:CP_Radial_D8.0mm_P3.50mm
- R11: value 2.7k -> 12k
- R12: value 1k -> 4.7k
Other:
- board text added: "V2.2"
- board text removed: "V2.1"
